Commit message: added some more basic packages

File: caato2_description/urdf/accessories/caato2.gazebo.xacro (robot description, xacro)
@@ -8,5 +8,5 @@
       <odometrySource>world</odometrySource>
       <publishOdomTF>true</publishOdomTF>
-      <robotBaseFrame>base_link</robotBaseFrame>
+      <robotBaseFrame>base_footprint</robotBaseFrame>
       <publishWheelTF>false</publishWheelTF>
       <publishTf>true</publishTf>

File: caato2_description/urdf/caato2.urdf.xacro (robot description, xacro)
@@ -36,4 +36,10 @@
     <origin rpy="0 0 0" xyz="0 0 0"/>
   </link>
+  <joint name="base_joint" type="fixed">
+    <origin xyz="0 0 ${wheel_radius}" rpy="0 0 0"/>
+    <parent link="base_footprint"/>
+    <child link="base_link"/>
+    <dynamics damping="0" friction="0"/>
+  </joint>
   <!-- Base link origin is at the centre of rotation of differential drive robot -->
   <link name="base_link">
@@ -51,4 +57,13 @@
       <material name="yellow"/>
     </visual>
+  <link name="imu_link">
+    <origin rpy="0 0 0" xyz="0 0 0"/>
+  </link>
+  <!-- In case of IMU -->
+    <joint name="imu_joint" type="fixed">
+      <parent link="base_link"/>
+      <child link="imu_link"/>
+      <origin xyz="0 0 0" rpy="0 0 0"/>
+    </joint>
   	<!-- Left Caster Wheel Visual -->
      <collision name="left_caster_wheel_collision">
@@ -96,10 +111,4 @@
     <minDepth>0.001</minDepth>
 </gazebo>
-  <joint name="base_joint" type="fixed">
-    <origin xyz="0 0 ${wheel_radius}" rpy="0 0 0"/>
-    <parent link="base_link"/>
-    <child link="base_footprint"/>
-    <dynamics damping="0" friction="0"/>
-  </joint>
   <link name="inertial_link" >
     <inertial>

Commit message: saving changes

File: caato2_description/urdf/accessories/caato2.gazebo.xacro (robot description, xacro)
@@ -63,5 +63,5 @@
   <gazebo reference="hokuyo_laser_scanner_1">
     <sensor type="ray" name="front_hokuyo_sensor">
-      <pose>0 0 0 0 0 0</pose>
+      <!-- <pose>0 0 0 0 0 0</pose> -->
       <visualize>false</visualize>
       <update_rate>10</update_rate>
@@ -86,5 +86,5 @@
       </ray>
       <plugin name="gazebo_ros_front_hokuyo_controller" filename="libgazebo_ros_laser.so">
-        <topicName>front_left/scan</topicName>
+        <topicName>front_right/scan</topicName>
         <frameName>hokuyo_laser_scanner_1</frameName>
       </plugin>
@@ -116,5 +116,5 @@
       </ray>
       <plugin name="gazebo_ros_back_hokuyo_controller" filename="libgazebo_ros_laser.so">
-        <topicName>back_right/scan</topicName>
+        <topicName>back_left/scan</topicName>
         <frameName>hokuyo_laser_scanner_2</frameName>
       </plugin>

File: caato2_description/urdf/accessories/sick_scan.urdf.xacro (robot description, xacro)
@@ -1,3 +1,4 @@
 <?xml version="1.0"?>
+<!-- currently not used in caato, was used in unodopo -->
 <robot xmlns:controller="http://playerstage.sourceforge.net/gazebo/xmlschema/#controller"
   xmlns:interface="http://playerstage.sourceforge.net/gazebo/xmlschema/#interface"

File: caato2_description/urdf/caato2.urdf.xacro (robot description, xacro)
@@ -37,5 +37,6 @@
   </link>
   <joint name="base_joint" type="fixed">
-    <origin xyz="0 0 ${wheel_radius}" rpy="0 0 0"/>
+  <!-- Rotated to match rviz config -->
+    <origin xyz="0 0 ${wheel_radius}" rpy="0 0 ${pi/2}"/>
     <parent link="base_footprint"/>
     <child link="base_link"/>
@@ -183,5 +184,5 @@
   <link name="hokuyo_laser_scanner_1">
     <visual>
-      <origin xyz="0 0 0" rpy="0 0 0" />
+      <origin xyz="0 0 -0.06" rpy="0 0 0" />
       <geometry>
         <mesh filename="package://caato2_description/meshes/sensors/hokuyo_laser_scanner.stl"/>
@@ -190,5 +191,5 @@
     </visual>
     <collision>
-      <origin xyz="0 0 0" rpy="0 0 0" />
+      <origin xyz="0 0 -0.06" rpy="0 0 0" />
       <geometry>
         <mesh filename="package://caato2_description/meshes/sensors/hokuyo_laser_scanner.stl"/>
@@ -199,5 +200,5 @@
     </collision>
     <inertial>
-      <origin xyz="0 0 0" rpy="0 0 0.785"/>
+      <origin xyz="0 0 -0.06" rpy="0 0 3.93"/>
       <mass value="0.2" />
       <inertia ixx="0" ixy="0"  ixz="0" iyy="0" iyz="0" izz="0" />
@@ -205,5 +206,5 @@
   </link>
 	<joint name="hokuyo_laser_scanner_1_joint" type="fixed">
-		<origin xyz="-0.210233 -0.262308 0.143200" rpy="0 0 0.785" />
+		<origin xyz="-0.210233 -0.262308 0.203200" rpy="0 0 3.93" />
 		<parent link="base_link" />
 		<child link="hokuyo_laser_scanner_1" />
@@ -213,5 +214,5 @@
   <link name="hokuyo_laser_scanner_2">
     <visual>
-      <origin xyz="0 0 0" rpy="0 0 0" />
+      <origin xyz="0 0 -0.06" rpy="0 0 0" />
       <geometry>
         <mesh filename="package://caato2_description/meshes/sensors/hokuyo_laser_scanner.stl"/>
@@ -220,5 +221,5 @@
     </visual>
     <collision>
-      <origin xyz="0 0 0" rpy="0 0 0" />
+      <origin xyz="0 0 -0.06" rpy="0 0 0" />
       <geometry>
         <mesh filename="package://caato2_description/meshes/sensors/hokuyo_laser_scanner.stl"/>
@@ -229,5 +230,5 @@
     </collision>
     <inertial>
-      <origin xyz="0 0 0" rpy="0 0 0.785"/>
+      <origin xyz="0 0 -0.06" rpy="0 0 0.785"/>
       <mass value="0.2" />
       <inertia ixx="0" ixy="0"  ixz="0" iyy="0" iyz="0" izz="0" />
@@ -235,5 +236,5 @@
   </link>
 	<joint name="hokuyo_laser_scanner_2_joint" type="fixed">
-		<origin xyz="0.213805 0.115872 0.143200" rpy="0 0 0.785" />
+		<origin xyz="0.213805 0.115872 0.203200" rpy="0 0 0.785" />
 		<parent link="base_link" />
 		<child link="hokuyo_laser_scanner_2" />

Commit message: fixed urdf, atc in progress

File: caato2_description/urdf/accessories/caato2.gazebo.xacro (robot description, xacro)
@@ -64,5 +64,5 @@
     <sensor type="ray" name="front_hokuyo_sensor">
       <!-- <pose>0 0 0 0 0 0</pose> -->
-      <visualize>false</visualize>
+      <visualize>true</visualize>
       <update_rate>10</update_rate>
       <ray>
@@ -94,5 +94,5 @@
     <sensor type="ray" name="back_hokuyo_sensor">
       <!-- <pose>0 0 0 0 0 0</pose> -->
-      <visualize>false</visualize>
+      <visualize>true</visualize>
       <update_rate>10</update_rate>
       <ray>

File: caato2_description/urdf/caato2.urdf.xacro (robot description, xacro)
@@ -48,6 +48,5 @@
     <origin rpy="0 0 0" xyz="0 0 0"/>
       <geometry>
-        <!-- <mesh filename="package://caato2_description/meshes/bases/Body.stl"/> -->
-        <box size="0.5 0.5 0.3" />
+        <mesh filename="package://caato2_description/meshes/bases/Body.stl"/>
       </geometry>
     </collision>
@@ -59,13 +58,4 @@
       <material name="yellow"/>
     </visual>
-  <link name="imu_link">
-    <origin rpy="0 0 0" xyz="0 0 0"/>
-  </link>
-  <!-- In case of IMU -->
-    <joint name="imu_joint" type="fixed">
-      <parent link="base_link"/>
-      <child link="imu_link"/>
-      <origin xyz="0 0 0" rpy="0 0 0"/>
-    </joint>
   	<!-- Left Caster Wheel Visual -->
      <collision name="left_caster_wheel_collision">
@@ -113,4 +103,22 @@
     <minDepth>0.001</minDepth>
 </gazebo>
+  <!-- In case of IMU -->
+  <link name="imu_link">
+    <origin rpy="0 0 0" xyz="0 0 0"/>
+  </link>
+  <joint name="imu_joint" type="fixed">
+    <parent link="base_link"/>
+    <child link="imu_link"/>
+    <origin xyz="0 0 0" rpy="0 0 0"/>
+  </joint>
+  <!-- for the sake of a box body, original stl blocking lidars -->
+  <link name="body_link">
+    <origin rpy="0 0 0" xyz="0 0 0"/>
+  </link>
+  <joint name="body_joint" type="fixed">
+    <parent link="base_link"/>
+    <child link="body_link"/>
+    <origin xyz="0 -0.05 0.14" rpy="0 0 0"/>
+  </joint>
   <link name="inertial_link" >
     <inertial>
@@ -191,13 +199,4 @@
       <material name="black"/>
     </visual>
-    <collision>
-      <origin xyz="0 0 -0.06" rpy="0 0 0" />
-      <geometry>
-        <mesh filename="package://caato2_description/meshes/sensors/hokuyo_laser_scanner.stl"/>
-      </geometry>
-      <material name="hokuyo_laser_scanner_material">
-        <color rgba="1 0.643137 0.0313725 1.0"/>
-      </material>
-    </collision>
     <inertial>
       <origin xyz="0 0 -0.06" rpy="0 0 3.93"/>
@@ -221,13 +220,4 @@
       <material name="black"/>
     </visual>
-    <collision>
-      <origin xyz="0 0 -0.06" rpy="0 0 0" />
-      <geometry>
-        <mesh filename="package://caato2_description/meshes/sensors/hokuyo_laser_scanner.stl"/>
-      </geometry>
-      <material name="hokuyo_laser_scanner_material">
-        <color rgba="1 0.643137 0.0313725 1.0"/>
-      </material>
-    </collision>
     <inertial>
       <origin xyz="0 0 -0.06" rpy="0 0 0.785"/>
@@ -243,8 +233,8 @@
 	</joint>
   <!-- front realsense sensor -->
-  <xacro:include filename="$(find realsense2_description)/urdf/_d435.front.urdf.xacro"/>
+  <xacro:include filename="$(find realsense2_description)/urdf/_d435.2.front.urdf.xacro"/>
   <xacro:include filename="$(find realsense2_description)/urdf/_d435.front.gazebo.xacro"/>
   <xacro:d435_front parent="base_link">
-      <origin xyz="-0 -0.35 0.232" rpy="0 0 -1.57" />
+      <origin xyz="-0 -0.34 0.235" rpy="0 0 -1.57" />
   </xacro:d435_front>
   <!-- back realsense sensor -->
@@ -252,5 +242,5 @@
   <xacro:include filename="$(find realsense2_description)/urdf/_d435.gazebo.xacro"/>
   <xacro:sensor_d435 parent="base_link">
-      <origin xyz="0 0.16 0.23" rpy="0 0 1.57" />
+      <origin xyz="0 0.15 0.235" rpy="0 0 1.57" />
   </xacro:sensor_d435>
 </robot>

Commit message: caato2 urdf with arm + lidars adjusted + costmap inflation reduced + navigation tuned abit

File: caato2_description/urdf/accessories/caato2.gazebo.xacro (robot description, xacro)
@@ -63,6 +63,5 @@
   <gazebo reference="hokuyo_laser_scanner_1">
     <sensor type="ray" name="front_hokuyo_sensor">
-      <!-- <pose>0 0 0 0 0 0</pose> -->
-      <visualize>false</visualize>
+      <visualize>true</visualize>
       <update_rate>10</update_rate>
       <ray>
@@ -93,6 +92,5 @@
   <gazebo reference="hokuyo_laser_scanner_2">
     <sensor type="ray" name="back_hokuyo_sensor">
-      <!-- <pose>0 0 0 0 0 0</pose> -->
-      <visualize>false</visualize>
+      <visualize>true</visualize>
       <update_rate>10</update_rate>
       <ray>
@@ -102,5 +100,6 @@
             <resolution>0.25</resolution>
             <min_angle>-2.356</min_angle>
-            <max_angle>2.356</max_angle>
+            <!-- accounting for the arm blocking -->
+            <max_angle>0.78</max_angle>
           </horizontal>
         </scan>

File: caato2_description/urdf/caato2.urdf.xacro (robot description, xacro)
@@ -46,13 +46,13 @@
   <link name="base_link">
     <collision name="collision_chassis">
-    <origin rpy="0 0 0" xyz="0 0 0"/>
-      <geometry>
-        <mesh filename="package://caato2_description/meshes/bases/Body.stl"/>
+      <origin rpy="0 0 0" xyz="0.08 0.172 0.182"/>
+      <geometry>
+        <mesh filename="package://caato2_description/meshes/bases/body_with_arm.stl"/>
       </geometry>
     </collision>
     <visual>
-    <origin rpy="0 0 0" xyz="0 0 0"/>
-      <geometry>
-        <mesh filename="package://caato2_description/meshes/bases/Body.stl"/>
+      <origin rpy="0 0 0" xyz="0.08 0.172 0.182"/>
+      <geometry>
+        <mesh filename="package://caato2_description/meshes/bases/body_with_arm.stl"/>
       </geometry>
       <material name="yellow"/>
@@ -236,5 +236,5 @@
   <xacro:include filename="$(find realsense2_description)/urdf/_d435.front.gazebo.xacro"/>
   <xacro:d435_front parent="base_link">
-      <origin xyz="-0 -0.34 0.235" rpy="0 0 -1.57" />
+      <origin xyz="-0 -0.34 0.46" rpy="0 0 -1.57" />
   </xacro:d435_front>
   <!-- back realsense sensor -->
@@ -242,5 +242,5 @@
   <xacro:include filename="$(find realsense2_description)/urdf/_d435.gazebo.xacro"/>
   <xacro:sensor_d435 parent="base_link">
-      <origin xyz="0 0.15 0.235" rpy="0 0 1.57" />
+      <origin xyz="0 0.197 0.46" rpy="0 0 1.57" />
   </xacro:sensor_d435>
 </robot>

Commit message: adjusted camera position by Abilash

File: caato2_description/urdf/accessories/caato2.gazebo.xacro (robot description, xacro)
@@ -76,5 +76,5 @@
         <range>
           <min>0.1</min>
-          <max>12</max>
+          <max>10</max>
         </range>
         <noise>
@@ -100,11 +100,10 @@
             <resolution>0.25</resolution>
             <min_angle>-2.356</min_angle>
-            <!-- accounting for the arm blocking -->
-            <max_angle>0.78</max_angle>
+            <max_angle>2.356</max_angle>
           </horizontal>
         </scan>
         <range>
           <min>0.1</min>
-          <max>12</max>
+          <max>10</max>
         </range>
         <noise>

File: caato2_description/urdf/caato2_3d.urdf.xacro (robot description, xacro)
@@ -236,5 +236,5 @@
   <xacro:include filename="$(find realsense2_description)/urdf/_d435.front.gazebo.xacro"/>
   <xacro:d435_front parent="base_link">
-      <origin xyz="-0 -0.34 0.46" rpy="0 0 -1.57" />
+      <origin xyz="-0 -0.34 0.35" rpy="0 0 -1.57" />
   </xacro:d435_front>
   <!-- back realsense sensor -->
@@ -242,5 +242,5 @@
   <xacro:include filename="$(find realsense2_description)/urdf/_d435.gazebo.xacro"/>
   <xacro:sensor_d435 parent="base_link">
-      <origin xyz="0 0.197 0.46" rpy="0 0 1.57" />
+      <origin xyz="0 0.28 0.46" rpy="0 0 1.57" />
   </xacro:sensor_d435>
   <!-- <xacro:include filename="$(find ouster_os1_64)/urdf/os1_64.urdf.xacro"/>
