Commit message: Updated /caato2_gazebo & caato2_description
Tightend eband_local_planner_params.yaml tolerances:
   xy_goal_tolerance: 0.1
   yaw_goal_tolerance: 0.05

File: caato2_description/urdf/common_properties.xacro (robot description, xacro)
@@ -1,6 +1,4 @@
 <?xml version="1.0" ?>
 <robot name="xacro_properties" xmlns:xacro="http://ros.org/wiki/xacro">
-  <!--degree to radians-->
-  <xacro:property name="pi" value="3.14259"/>
   <!-- Init colour -->
   <material name="black">
