Commit message: tuned inertial values, center of mass and damping and friction values

File: caato2_description/urdf/caato2.urdf.xacro (robot description, xacro)
@@ -6,5 +6,5 @@
   <xacro:property name="base_depth" value="0.52" />
   <xacro:property name="base_height" value="0.37" />
-  <xacro:property name="base_mass" value="5" />
+  <xacro:property name="base_mass" value="46.143" />
   <!-- Wheel Mounting Positions -->
   <xacro:property name="wheelbase" value="NA since differential drive" />
@@ -70,6 +70,8 @@
       <mass value="${base_mass}" />
       <!--shifted weight to prevent jerking-->
-      <origin xyz="0 0.011 0"/>
-      <xacro:cuboid_inertia m="${base_mass}" w="${base_width}" h="${base_height}" d="${base_depth}"/>
+      <origin xyz="0 -0.120 0.045"/>
+      <inertia ixx="1.291" ixy = "0" ixz = "0"
+                iyy="1.381" iyz = "0"
+                izz="1.976" />
     </inertial>
   </link>
@@ -161,5 +163,5 @@
     <axis rpy="0 0 0" xyz="0 0 1"/>
     <limit effort="10000" velocity="1000"/>
-    <dynamics damping="0" friction="0.0"/>
+    <dynamics damping="0.5" friction="0.5"/>
   </joint>
     <!-- Right caster wheel -->
@@ -189,5 +191,5 @@
     <axis rpy="0 0 0" xyz="0 0 1"/>
     <limit effort="10000" velocity="1000"/>
-    <dynamics damping="0" friction="0.0"/>
+    <dynamics damping="0.5" friction="0.5"/>
   </joint>
   <!-- Lider Sensor 1_Front -->

Commit message: more tuning

File: caato2_description/urdf/caato2.urdf.xacro (robot description, xacro)
@@ -137,4 +137,8 @@
     <dynamics damping="0" friction="1.0"/>
   </joint>
+  <!-- Caster wheel damping and friction macro-->
+  <xacro:macro name="caster_wheel_swivel_joint_damping_friction">
+        <dynamics damping="0.05" friction="0.2"/>
+    </xacro:macro>
   <!-- Left caster wheel -->
   <link name="left_caster_wheel_link">
@@ -163,5 +167,5 @@
     <axis rpy="0 0 0" xyz="0 0 1"/>
     <limit effort="10000" velocity="1000"/>
-    <dynamics damping="0.5" friction="0.5"/>
+    <xacro:caster_wheel_swivel_joint_damping_friction />
   </joint>
     <!-- Right caster wheel -->
@@ -191,5 +195,5 @@
     <axis rpy="0 0 0" xyz="0 0 1"/>
     <limit effort="10000" velocity="1000"/>
-    <dynamics damping="0.5" friction="0.5"/>
+    <xacro:caster_wheel_swivel_joint_damping_friction />
   </joint>
   <!-- Lider Sensor 1_Front -->

Commit message: edited casters to be part of chassis

File: caato2_description/urdf/caato2.urdf.xacro (robot description, xacro)
@@ -51,4 +51,40 @@
       <material name="yellow"/>
     </visual>
+  	<!-- Left Caster Wheel Visual -->
+     <collision name="left_caster_wheel_collision">
+      <origin xyz="0.184979 -0.22 -0.0516" rpy="0 0 0"/>
+      <geometry>
+        <sphere radius="${caster_wheel_radius}"/>
+      </geometry>
+      <surface>
+        <friction>
+          <ode>
+            <mu>0</mu>
+            <mu2>0</mu2>
+            <slip1>1.0</slip1>
+            <slip2>1.0</slip2>
+          </ode>
+        </friction>
+      </surface>
+    </collision>
+    <visual name="left_caster_wheel_visual">
+      <origin xyz="0.184979 -0.22 0.0484" rpy="0 0 1.2"/>
+      <geometry>
+        <mesh filename="package://caato2_description/meshes/wheels/caster_wheel.stl"/>
+      </geometry>
+    </visual>
+    <!-- Right Caster Wheel Visual -->
+    <collision name="right_caster_wheel_collision">
+    <origin xyz="-0.184979 -0.22 -0.0516" rpy="0 0 0"/>
+      <geometry>
+        <sphere radius="${caster_wheel_radius}"/>
+      </geometry>
+    </collision>
+    <visual name="right_caster_wheel_visual">
+      <origin xyz="-0.184979 -0.22 0.0484" rpy="0 0 1.2"/>
+      <geometry>
+        <mesh filename="package://caato2_description/meshes/wheels/caster_wheel.stl"/>
+      </geometry>
+    </visual>
   </link>
   <gazebo reference="base_link">
@@ -69,6 +105,6 @@
     <inertial>
       <mass value="${base_mass}" />
-      <!--shifted weight to prevent jerking-->
-      <origin xyz="0 0.011 0"/>
+      <!--shifted weight if needed to prevent jerking-->
+      <origin xyz="0 0 -0.13"/>
       <xacro:cuboid_inertia m="${base_mass}" w="${base_width}" h="${base_height}" d="${base_depth}"/>
     </inertial>
@@ -134,60 +170,4 @@
     <limit effort="10000" velocity="1000"/>
     <dynamics damping="0" friction="1.0"/>
-  </joint>
-  <!-- Left caster wheel -->
-  <link name="left_caster_wheel_link">
-    <inertial>
-      <mass value="${caster_wheel_mass}"/>
-      <origin xyz="0 0 0" rpy="0 0 0"/>
-      <xacro:cylinder_inertia m="${caster_wheel_mass}" r="${caster_wheel_radius}" h="${caster_wheel_width}" />
-    </inertial>
-    <collision name="left_caster_wheel_collision">
-      <origin xyz="0 0 -0.1" rpy="0 0 0"/>
-      <geometry>
-        <sphere radius="${caster_wheel_radius}"/>
-      </geometry>
-    </collision>
-    <visual name="left_caster_wheel_visual">
-      <origin xyz="0 0 0" rpy="0 0 0"/>
-      <geometry>
-        <mesh filename="package://caato2_description/meshes/wheels/caster_wheel.stl"/>
-      </geometry>
-    </visual>
-  </link>
-  <joint name="left_caster_wheel_joint" type="continuous">
-    <origin xyz="0.184979 -0.22 0.0484" rpy="0 0 0"/>
-    <child link="left_caster_wheel_link"/>
-    <parent link="base_link"/>
-    <axis rpy="0 0 0" xyz="0 0 1"/>
-    <limit effort="10000" velocity="1000"/>
-    <dynamics damping="0" friction="0.0"/>
-  </joint>
-    <!-- Right caster wheel -->
-  <link name="right_caster_wheel_link">
-    <inertial>
-      <mass value="${caster_wheel_mass}"/>
-      <origin xyz="0 0 0" rpy="0 0 0"/>
-      <xacro:cylinder_inertia m="${caster_wheel_mass}" r="${caster_wheel_radius}" h="${caster_wheel_width}" />
-    </inertial>
-    <collision name="right_caster_wheel_collision">
-      <origin xyz="0 0 -0.1" rpy="0 0 0"/>
-      <geometry>
-        <sphere radius="${caster_wheel_radius}"/>
-      </geometry>
-    </collision>
-    <visual name="right_caster_wheel_visual">
-      <origin xyz="0 0 0" rpy="0 0 0"/>
-      <geometry>
-        <mesh filename="package://caato2_description/meshes/wheels/caster_wheel.stl"/>
-      </geometry>
-    </visual>
-  </link>
-  <joint name="right_caster_wheel_joint" type="continuous">
-    <origin xyz="-0.184979 -0.22 0.0484" rpy="0 0 0"/>
-    <child link="right_caster_wheel_link"/>
-    <parent link="base_link"/>
-    <axis rpy="0 0 0" xyz="0 0 1"/>
-    <limit effort="10000" velocity="1000"/>
-    <dynamics damping="0" friction="0.0"/>
   </joint>
   <!-- Lider Sensor 1_Front -->

Commit message: revert back to unmerged

File: caato2_description/urdf/caato2.urdf.xacro (robot description, xacro)
@@ -105,9 +105,7 @@
     <inertial>
       <mass value="${base_mass}" />
-      <!--shifted weight to prevent jerking-->
-      <origin xyz="0 -0.120 0.045"/>
-      <inertia ixx="1.291" ixy = "0" ixz = "0"
-                iyy="1.381" iyz = "0"
-                izz="1.976" />
+      <!--shifted weight if needed to prevent jerking-->
+      <origin xyz="0 0 -0.13"/>
+      <xacro:cuboid_inertia m="${base_mass}" w="${base_width}" h="${base_height}" d="${base_depth}"/>
     </inertial>
   </link>
@@ -172,64 +170,4 @@
     <limit effort="10000" velocity="1000"/>
     <dynamics damping="0" friction="1.0"/>
-  </joint>
-  <!-- Caster wheel damping and friction macro-->
-  <xacro:macro name="caster_wheel_swivel_joint_damping_friction">
-        <dynamics damping="0.05" friction="0.2"/>
-    </xacro:macro>
-  <!-- Left caster wheel -->
-  <link name="left_caster_wheel_link">
-    <inertial>
-      <mass value="${caster_wheel_mass}"/>
-      <origin xyz="0 0 0" rpy="0 0 0"/>
-      <xacro:cylinder_inertia m="${caster_wheel_mass}" r="${caster_wheel_radius}" h="${caster_wheel_width}" />
-    </inertial>
-    <collision name="left_caster_wheel_collision">
-      <origin xyz="0 0 -0.1" rpy="0 0 0"/>
-      <geometry>
-        <sphere radius="${caster_wheel_radius}"/>
-      </geometry>
-    </collision>
-    <visual name="left_caster_wheel_visual">
-      <origin xyz="0 0 0" rpy="0 0 0"/>
-      <geometry>
-        <mesh filename="package://caato2_description/meshes/wheels/caster_wheel.stl"/>
-      </geometry>
-    </visual>
-  </link>
-  <joint name="left_caster_wheel_joint" type="continuous">
-    <origin xyz="0.184979 -0.22 0.0484" rpy="0 0 0"/>
-    <child link="left_caster_wheel_link"/>
-    <parent link="base_link"/>
-    <axis rpy="0 0 0" xyz="0 0 1"/>
-    <limit effort="10000" velocity="1000"/>
-    <xacro:caster_wheel_swivel_joint_damping_friction />
-  </joint>
-    <!-- Right caster wheel -->
-  <link name="right_caster_wheel_link">
-    <inertial>
-      <mass value="${caster_wheel_mass}"/>
-      <origin xyz="0 0 0" rpy="0 0 0"/>
-      <xacro:cylinder_inertia m="${caster_wheel_mass}" r="${caster_wheel_radius}" h="${caster_wheel_width}" />
-    </inertial>
-    <collision name="right_caster_wheel_collision">
-      <origin xyz="0 0 -0.1" rpy="0 0 0"/>
-      <geometry>
-        <sphere radius="${caster_wheel_radius}"/>
-      </geometry>
-    </collision>
-    <visual name="right_caster_wheel_visual">
-      <origin xyz="0 0 0" rpy="0 0 0"/>
-      <geometry>
-        <mesh filename="package://caato2_description/meshes/wheels/caster_wheel.stl"/>
-      </geometry>
-    </visual>
-  </link>
-  <joint name="right_caster_wheel_joint" type="continuous">
-    <origin xyz="-0.184979 -0.22 0.0484" rpy="0 0 0"/>
-    <child link="right_caster_wheel_link"/>
-    <parent link="base_link"/>
-    <axis rpy="0 0 0" xyz="0 0 1"/>
-    <limit effort="10000" velocity="1000"/>
-    <xacro:caster_wheel_swivel_joint_damping_friction />
   </joint>
   <!-- Lider Sensor 1_Front -->

Commit message: update

File: caato2_description/urdf/caato2.urdf.xacro (robot description, xacro)
@@ -241,3 +241,15 @@
 		<axis xyz="0 0 1"/>
 	</joint>
+  <!-- front realsense sensor -->
+  <xacro:include filename="$(find realsense2_description)/urdf/_d435.front.urdf.xacro"/>
+  <xacro:include filename="$(find realsense2_description)/urdf/_d435.front.gazebo.xacro"/>
+  <xacro:d435_front parent="base_link">
+      <origin xyz="-0 -0.35 0.232" rpy="0 0 -1.57" />
+  </xacro:d435_front>
+  <!-- back realsense sensor -->
+  <xacro:include filename="$(find realsense2_description)/urdf/_d435.2.urdf.xacro"/>
+  <xacro:include filename="$(find realsense2_description)/urdf/_d435.gazebo.xacro"/>
+  <xacro:sensor_d435 parent="base_link">
+      <origin xyz="0 0.16 0.23" rpy="0 0 1.57" />
+  </xacro:sensor_d435>
 </robot>

Commit message: fixed weird lidar scan thing, changed caato2 body collision to box

File: caato2_description/urdf/caato2.urdf.xacro (robot description, xacro)
@@ -48,5 +48,6 @@
     <origin rpy="0 0 0" xyz="0 0 0"/>
       <geometry>
-        <mesh filename="package://caato2_description/meshes/bases/Body.stl"/>
+        <!-- <mesh filename="package://caato2_description/meshes/bases/Body.stl"/> -->
+        <box size="0.5 0.5 0.3" />
       </geometry>
     </collision>

Commit message: new trl mod

File: caato2_description/urdf/caato2.urdf.xacro (robot description, xacro)
@@ -236,5 +236,5 @@
   <xacro:include filename="$(find realsense2_description)/urdf/_d435.front.gazebo.xacro"/>
   <xacro:d435_front parent="base_link">
-      <origin xyz="-0 -0.34 0.46" rpy="0 0 -1.57" />
+      <origin xyz="-0 -0.34 0.35" rpy="0 0 -1.57" />
   </xacro:d435_front>
   <!-- back realsense sensor -->
@@ -242,5 +242,5 @@
   <xacro:include filename="$(find realsense2_description)/urdf/_d435.gazebo.xacro"/>
   <xacro:sensor_d435 parent="base_link">
-      <origin xyz="0 0.197 0.46" rpy="0 0 1.57" />
+      <origin xyz="0 0.28 0.46" rpy="0 0 1.57" />
   </xacro:sensor_d435>
 </robot>

Commit message: Solved some bugs
Increased the e-band gains significantly, resulting in tighter capture
tolerances

File: caato2_description/urdf/caato2.urdf.xacro (robot description, xacro)
@@ -38,5 +38,5 @@
   <joint name="base_joint" type="fixed">
   <!-- Rotated to match rviz config -->
-    <origin xyz="0 0 ${wheel_radius}" rpy="0 0 ${pi/2}"/>
+    <origin xyz="-0.0 0 ${wheel_radius}" rpy="0 0 ${pi/2}"/>
     <parent link="base_footprint"/>
     <child link="base_link"/>
